File: PneumaticValveController.kicad_pcb (KiCad board)
At the start: 4 copper layers, 101.6 x 67.5 mm, 81 parts, among them IC10 PS7, IC2 L7805ABD2T-TR, IC3 PS1, IC4 PS2, IC5 PS4, IC6 PS3, IC7 PS5, IC8 PS6, IC9 PS8, J1 Power, J10 PUMP3, J11 PUMP4, J12 PUMP5, J13 PUMP6, J14 PUMP7, J15 PUMP8, J16 SOL1, J17 SOL3, J18 SOL2, J19 SOL4, J2 PWM, J20 SOL5, J21 SOL7, J22 SOL6, J23 SOL8, J24 Barrel_Jack, J3 Analog, J4 PWM, J5 Analog, J6 Communication, J7 Digital, J8 PUMP1, J9 PUMP2, Q1 IRFR320TRPBF-BE3, Q2 IRFR320TRPBF-BE3, Q3 IRFR320TRPBF-BE3, Q4 IRFR320TRPBF-BE3, Q5 IRFR320TRPBF-BE3, Q6 IRFR320TRPBF-BE3, Q7 IRFR320TRPBF-BE3, Q8 IRFR320TRPBF-BE3, U1 TXS0108EPW, U2 TXS0108EPW

Commit message: Add files via upload
Chnges 11/15/2022
Parts:
- G***: value LOGO -> CHARMLAB
- moved G*** 14.5 mm to (120.3, 96.8), turned to 0 degrees
- moved J24 1.52 mm to (114.5, 89.2)
Routing:
- net /PneumaticsAndConnectors/SOL1: track 105.1 -> 94.3 mm
- net +12V: track 12.3 -> 13.6 mm
- net /Pump/PUMP1_PWM_5: track 45.0 -> 43.9 mm
Other:
- board text added: "Electro-Pneumatic Controller"
- board text added: "S. Wallace Z. Zhakypov 2022"
- board text removed: "Voxel Controller"
- board text removed: "Z. Zhakypov, S. Wallace"
